Commit message: ROS2 SwiftPro 可視化修復與問題記錄
- 添加URDF碰撞幾何到所有鏈接
- 修改RViz配置使用基本RobotModel顯示
- 添加靜態變換發布器
- 詳細記錄當前問題和解決方案
- 更新README包含完整問題分析和開發計劃

File: swiftpro/urdf/pro_model.urdf (robot description, URDF)
Before this commit: robot swiftpro, 10 links, 9 joints
Links:
- link Base: geometry visual mesh filename=package://swiftpro/urdf/pro_links/Base.STL
- link Link1: geometry visual mesh filename=package://swiftpro/urdf/pro_links/Link1.STL
- link Link2: geometry visual mesh filename=package://swiftpro/urdf/pro_links/Link2.STL
- link Link3: geometry visual mesh filename=package://swiftpro/urdf/pro_links/Link3.STL
- link Link4: geometry visual mesh filename=package://swiftpro/urdf/pro_links/Link4.STL
- link Link5: geometry visual mesh filename=package://swiftpro/urdf/pro_links/Link5.STL
- link Link6: geometry visual mesh filename=package://swiftpro/urdf/pro_links/Link6.STL
- link Link7: geometry visual mesh filename=package://swiftpro/urdf/pro_links/Link7.STL
- link Link8: geometry visual mesh filename=package://swiftpro/urdf/pro_links/Gripper.STL
- link Link9: geometry visual mesh filename=package://swiftpro/urdf/pro_links/Link9.STL
